File: kicad/DeauthGeiger.kicad_sch (KiCad schematic)
At the start: 4 parts, among them SW1 Reset, U2 ESP32-C3

Commit message: sync
Parts:
- removed AE1: Antenna, symbol Device:Antenna
- added C1, C2: C, symbol Device:C
- added J1: Conn_Coaxial_Small, symbol Connector:Conn_Coaxial_Small
- added R2: R, symbol Device:R
- added Y1: Crystal_GND24, symbol Device:Crystal_GND24
Connections:
- net GND: now also U2.33 (GND), C1.2, C2.2
- net at U2.1 (LNA_IN): now also J1.1 (In)
- net at U2.29 (XTAL_N): now also Y1.1
- net at U2.30 (XTAL_P): now also R2.2
- net GPIO0: now reaches U2.4 (XTAL_32K_P)
- net GPIO1: now reaches U2.5 (XTAL_32K_N)
- new net: C2.1, Y1.4
- new net: C1.1, Y1.2
- new net: R2.1, Y1.3

Commit message: sync
Parts:
- added J2: USB_C_Receptacle_USB2.0_16P, symbol Connector:USB_C_Receptacle_USB2.0_16P
- added R3, R4: 10k, Resistor_SMD:R_0603_1608Metric, symbol Device:R
- added R5, R6: 10k, symbol Device:R
- added SW2: SCAN/HOLD, symbol Switch:SW_SPST
- added SW3: RotaryEncoder_Switch_MP, Rotary_Encoder:RotaryEncoder_Alps_EC12E-Switch_Vertical_H20mm, symbol Device:RotaryEncoder_Switch_MP
- C1, C2: footprint (none) -> Capacitor_SMD:C_0603_1608Metric
- R1, R2: footprint (none) -> Resistor_SMD:R_0603_1608Metric
- Y1: value Crystal_GND24 -> 160MHz
Connections:
- net +3V3: now also U2.11 (VDD3P3_RTC), U2.17 (VDD3P3_CPU), U2.2 (VDD3P3), U2.3 (VDD3P3), SW3.C
- net GND: now also J1.2 (Ext), J2.A1 (GND), J2.A12 (GND), J2.B1 (GND), J2.B12 (GND), J2.S1 (SHIELD), R3.1, R4.1, R5.1, R6.2, SW3.MP
- net USB-D-: now reaches U2.25 (GPIO18)
- net USB-D-: now also J2.A7 (D-), J2.B7 (D-)
- net USB-D+: now reaches U2.26 (GPIO19)
- net USB-D+: now also J2.A6 (D+), J2.B6 (D+)
- new net: R3.2, SW3.B
- new net: R4.2, SW3.A
- new net: J2.A8 (SBU1), J2.B8 (SBU2), R6.1
- new net: J2.A5 (CC1), J2.B5 (CC2), R5.2
- new net +5V: J2.A4 (VBUS), J2.A9 (VBUS), J2.B4 (VBUS), J2.B9 (VBUS)
Other:
- moved on the sheet: J1

Commit message: sync
Parts:
- added LS1: Speaker, symbol Device:Speaker
- added MES1: Strength, symbol Device:Voltmeter_DC
- added U1: CR2013-MI2120, Display:CR2013-MI2120, symbol Driver_Display:CR2013-MI2120
Connections:
- net GND: now also LS1.2, MES1.1 (-)
